Commit message: update 1

File: model_generator_hrc/phonebot_general.urdf (robot description, URDF)
Before this commit: robot phonebot_general_6motor, 28 links, 27 joints
Joints:
- joint l_ankle_pitch_joint: origin xyz=0.000000 -0.100000 0.000000 rpy=0.000000 0.000000 3.141593 -> xyz=0.000000 -0.110000 0.000000 rpy=0.000000 0.000000 3.141593
- joint r_ankle_pitch_joint: origin xyz=-0.000000 -0.100000 0.000000 rpy=0.000000 -0.000000 -3.141593 -> xyz=-0.000000 -0.110000 0.000000 rpy=0.000000 -0.000000 -3.141593
