Commit message: good version v2

File: model_generator_hrc/chopstick_bot_general.urdf (robot description, URDF)
Before this commit: robot chopstick_bot, 12 links, 11 joints
Links:
- removed link l_hip_pitch_joint_frame
- removed link l_hip_pitch_mount
- removed link l_leg_bar
- removed link r_hip_pitch_joint_frame
- removed link r_hip_pitch_mount
- removed link r_leg_bar
- added link l_end_effector, mass 0.030000; collision cylinder length=0.200000 radius=0.005000; visual cylinder length=0.200000 radius=0.005000
- added link l_hip_pitch_out
- added link l_hip_roll_out
- added link r_end_effector, mass 0.030000; collision cylinder length=0.200000 radius=0.005000; visual cylinder length=0.200000 radius=0.005000
- added link r_hip_pitch_out
- added link r_hip_roll_out
Joints:
- removed joint base_to_l_hip_pitch_mount_fixed
- removed joint base_to_r_hip_pitch_mount_fixed
- removed joint l_hip_pitch_mount_to_motor_fixed
- removed joint l_hip_pitch_to_l_hip_roll_fixed
- removed joint r_hip_pitch_mount_to_motor_fixed
- removed joint r_hip_pitch_to_r_hip_roll_fixed
- added joint l_end_effector_fixed: type fixed, parent l_hip_roll_out, child l_end_effector, origin xyz=0.000000 -0.170000 0.000000 rpy=0.000000 0.000000 0.000000
- added joint l_hip_pitch_mount_fixed: type fixed, parent base_motor_link, child l_hip_pitch, origin xyz=-0.040000 0.000000 0.000000 rpy=0.000000 -1.570796 0.000000
- added joint l_hip_roll_mount_fixed: type fixed, parent l_hip_pitch_out, child l_hip_roll, origin xyz=0.000000 0.000000 0.040000 rpy=0.000000 -1.570796 -1.570796
- added joint r_end_effector_fixed: type fixed, parent r_hip_roll_out, child r_end_effector, origin xyz=-0.000000 -0.170000 0.000000 rpy=0.000000 -0.000000 0.000000
- added joint r_hip_pitch_mount_fixed: type fixed, parent base_motor_link, child r_hip_pitch, origin xyz=0.040000 0.000000 0.000000 rpy=0.000000 1.570796 -0.000000
- added joint r_hip_roll_mount_fixed: type fixed, parent r_hip_pitch_out, child r_hip_roll, origin xyz=-0.000000 0.000000 0.040000 rpy=0.000000 1.570796 1.570796
- joint l_hip_pitch_joint: child l_hip_pitch_joint_frame -> l_hip_pitch_out; limit lower=-1.57 upper=1.57 effort=3.0 velocity=6.0 -> lower=-3.14159 upper=3.14159 effort=5.0 velocity=8.0; origin xyz=0.000000 0.000000 0.040000 rpy=0.000000 0.000000 0.000000 -> xyz=0.000000 0.000000 0.000000 rpy=0.000000 0.000000 0.000000
- joint l_hip_roll_joint: child l_leg_bar -> l_hip_roll_out; limit lower=-1.57 upper=1.57 effort=3.0 velocity=6.0 -> lower=-3.14159 upper=3.14159 effort=5.0 velocity=8.0; origin xyz=0.000000 -0.000000 0.000000 rpy=0.000000 0.000000 0.000000 -> xyz=0.000000 0.000000 0.000000 rpy=0.000000 0.000000 0.000000
- joint r_hip_pitch_joint: child r_hip_pitch_joint_frame -> r_hip_pitch_out; limit lower=-1.57 upper=1.57 effort=3.0 velocity=6.0 -> lower=-3.14159 upper=3.14159 effort=5.0 velocity=8.0; origin xyz=-0.000000 0.000000 0.040000 rpy=0.000000 0.000000 0.000000 -> xyz=0.000000 0.000000 0.000000 rpy=0.000000 0.000000 0.000000
- joint r_hip_roll_joint: child r_leg_bar -> r_hip_roll_out; limit lower=-1.57 upper=1.57 effort=3.0 velocity=6.0 -> lower=-3.14159 upper=3.14159 effort=5.0 velocity=8.0; origin xyz=-0.000000 -0.000000 0.000000 rpy=0.000000 0.000000 0.000000 -> xyz=0.000000 0.000000 0.000000 rpy=0.000000 0.000000 0.000000

File: model_generator_hrc/phonebot_general.urdf (robot description, URDF)
Before this commit: robot phonebot, 28 links, 27 joints
Links:
- removed link l_ankle_pitch_joint_frame
- removed link l_ankle_roll_joint_frame
- removed link l_foot
- removed link l_hip_calf_joint_frame
- removed link l_hip_pitch_mount
- removed link l_hip_roll_joint_frame
- removed link l_hip_thigh_joint_frame
- removed link r_ankle_pitch_joint_frame
- removed link r_ankle_roll_joint_frame
- removed link r_foot
- removed link r_hip_calf_joint_frame
- removed link r_hip_pitch_mount
- removed link r_hip_roll_joint_frame
- removed link r_hip_thigh_joint_frame
- added link l_ankle_pitch_out, mass 0.001000
- added link l_ankle_roll_out, mass 0.001000
- added link l_end_effector, mass 0.050000; collision box size=0.100000 0.060000 0.010000; visual box size=0.100000 0.060000 0.010000
- added link l_hip_calf_out, mass 0.001000
- added link l_hip_pitch_out, mass 0.001000
- added link l_hip_roll_out, mass 0.001000
- added link l_hip_thigh_out, mass 0.001000
- added link r_ankle_pitch_out, mass 0.001000
- added link r_ankle_roll_out, mass 0.001000
- added link r_end_effector, mass 0.050000; collision box size=0.100000 0.060000 0.010000; visual box size=0.100000 0.060000 0.010000
- added link r_hip_calf_out, mass 0.001000
- added link r_hip_pitch_out, mass 0.001000
- added link r_hip_roll_out, mass 0.001000
- added link r_hip_thigh_out, mass 0.001000
Joints:
- removed joint base_to_l_hip_pitch_mount_fixed
- removed joint base_to_r_hip_pitch_mount_fixed
- removed joint l_ankle_pitch_joint_frame_to_motor_fixed
- removed joint l_ankle_roll_joint_frame_to_motor_fixed
- removed joint l_ankle_roll_to_l_foot_fixed
- removed joint l_hip_calf_joint_frame_to_motor_fixed
- removed joint l_hip_pitch_mount_to_motor_fixed
- removed joint r_ankle_pitch_joint_frame_to_motor_fixed
- removed joint r_ankle_roll_joint_frame_to_motor_fixed
- removed joint r_ankle_roll_to_r_foot_fixed
- removed joint r_hip_calf_joint_frame_to_motor_fixed
- removed joint r_hip_pitch_mount_to_motor_fixed
- added joint l_ankle_pitch_to_out_fixed: type fixed, parent l_ankle_pitch, child l_ankle_pitch_out, origin xyz=0.000000 0.000000 0.000000 rpy=0.000000 0.000000 0.000000
- added joint l_ankle_roll_mount_fixed: type fixed, parent l_ankle_pitch_out, child l_ankle_roll, origin xyz=-0.040000 0.000000 0.000000 rpy=0.000000 1.570796 0.000000
- added joint l_end_effector_fixed: type fixed, parent l_ankle_roll_out, child l_end_effector, origin xyz=0.000000 0.035000 0.040000 rpy=1.570796 -1.570796 0.000000
- added joint l_hip_calf_to_out_fixed: type fixed, parent l_hip_calf, child l_hip_calf_out, origin xyz=0.000000 0.000000 0.000000 rpy=0.000000 0.000000 0.000000
- added joint l_hip_pitch_joint: type revolute, parent l_hip_pitch, child l_hip_pitch_out, origin xyz=0.000000 0.000000 0.000000 rpy=0.000000 0.000000 0.000000, axis 0.000000 0.000000 1.000000, limit lower=-3.14159 upper=3.14159 effort=5.0 velocity=8.0
- added joint l_hip_pitch_mount_fixed: type fixed, parent base_motor_link, child l_hip_pitch, origin xyz=-0.050000 0.000000 0.000000 rpy=0.000000 -1.570796 0.000000
- added joint r_ankle_pitch_to_out_fixed: type fixed, parent r_ankle_pitch, child r_ankle_pitch_out, origin xyz=0.000000 0.000000 0.000000 rpy=0.000000 0.000000 0.000000
- added joint r_ankle_roll_mount_fixed: type fixed, parent r_ankle_pitch_out, child r_ankle_roll, origin xyz=0.040000 0.000000 0.000000 rpy=0.000000 -1.570796 -0.000000
- added joint r_end_effector_fixed: type fixed, parent r_ankle_roll_out, child r_end_effector, origin xyz=-0.000000 0.035000 0.040000 rpy=0.000000 1.570796 -1.570796
- added joint r_hip_calf_to_out_fixed: type fixed, parent r_hip_calf, child r_hip_calf_out, origin xyz=0.000000 0.000000 0.000000 rpy=0.000000 0.000000 0.000000
- added joint r_hip_pitch_joint: type revolute, parent r_hip_pitch, child r_hip_pitch_out, origin xyz=0.000000 0.000000 0.000000 rpy=0.000000 0.000000 0.000000, axis 0.000000 0.000000 1.000000, limit lower=-3.14159 upper=3.14159 effort=5.0 velocity=8.0
- added joint r_hip_pitch_mount_fixed: type fixed, parent base_motor_link, child r_hip_pitch, origin xyz=0.050000 0.000000 0.000000 rpy=0.000000 1.570796 -0.000000
- joint l_ankle_pitch_joint: child l_ankle_pitch_joint_frame -> l_ankle_pitch; origin xyz=0.000000 -0.100000 0.000000 rpy=0.000000 0.000000 0.000000 -> xyz=0.000000 -0.100000 0.000000 rpy=0.000000 0.000000 3.141593; parent l_hip_calf -> l_hip_calf_out
- joint l_ankle_roll_joint: child l_ankle_roll_joint_frame -> l_ankle_roll_out; origin xyz=-0.040000 0.000000 0.000000 rpy=0.000000 0.000000 0.000000 -> xyz=0.000000 0.000000 0.000000 rpy=0.000000 0.000000 0.000000; parent l_ankle_pitch -> l_ankle_roll
- joint l_hip_calf_joint: child l_hip_calf_joint_frame -> l_hip_calf; origin xyz=0.000000 0.000000 0.040000 rpy=0.000000 0.000000 0.000000 -> xyz=0.000000 0.000000 0.040000 rpy=-1.570796 0.000000 -1.570796; parent l_hip_thigh_joint_frame -> l_hip_thigh_out
- joint l_hip_roll_joint: child l_hip_roll_joint_frame -> l_hip_roll_out
- joint l_hip_roll_mount_fixed: parent l_hip_pitch -> l_hip_pitch_out
- joint l_hip_thigh_joint: child l_hip_thigh_joint_frame -> l_hip_thigh_out
- joint l_hip_thigh_mount_fixed: parent l_hip_roll_joint_frame -> l_hip_roll_out
- joint r_ankle_pitch_joint: child r_ankle_pitch_joint_frame -> r_ankle_pitch; origin xyz=-0.000000 -0.100000 0.000000 rpy=0.000000 0.000000 0.000000 -> xyz=-0.000000 -0.100000 0.000000 rpy=0.000000 -0.000000 -3.141593; parent r_hip_calf -> r_hip_calf_out
- joint r_ankle_roll_joint: child r_ankle_roll_joint_frame -> r_ankle_roll_out; origin xyz=0.040000 0.000000 0.000000 rpy=0.000000 0.000000 0.000000 -> xyz=0.000000 0.000000 0.000000 rpy=0.000000 0.000000 0.000000; parent r_ankle_pitch -> r_ankle_roll
- joint r_hip_calf_joint: child r_hip_calf_joint_frame -> r_hip_calf; origin xyz=-0.000000 0.000000 0.040000 rpy=0.000000 0.000000 0.000000 -> xyz=-0.000000 0.000000 0.040000 rpy=-1.570796 -0.000000 1.570796; parent r_hip_thigh_joint_frame -> r_hip_thigh_out
- joint r_hip_roll_joint: child r_hip_roll_joint_frame -> r_hip_roll_out
- joint r_hip_roll_mount_fixed: parent r_hip_pitch -> r_hip_pitch_out
- joint r_hip_thigh_joint: child r_hip_thigh_joint_frame -> r_hip_thigh_out
- joint r_hip_thigh_mount_fixed: parent r_hip_roll_joint_frame -> r_hip_roll_out

Commit message: good v2

File: model_generator_hrc/chopstick_bot_general.urdf (robot description, URDF)
Before this commit: robot chopstick_bot, 12 links, 11 joints
Links:
- link l_hip_pitch_out: mass None -> 0.001000
- link l_hip_roll_out: mass None -> 0.001000
- link r_hip_pitch_out: mass None -> 0.001000
- link r_hip_roll_out: mass None -> 0.001000

Commit message: good version for model generate

File: model_generator_hrc/chopstick_bot_general.urdf (robot description, URDF)
Before this commit: robot chopstick_bot, 12 links, 11 joints
Links:
- link base_motor_link: geometry collision box size=0.028500 0.046500 0.034000; visual mesh filename=meshes/XL-430_new_coordinate_on_axis.STL scale=0.001000 0.001000 0.001000
- link l_hip_pitch: geometry collision box size=0.028500 0.046500 0.034000; visual mesh filename=meshes/XL-430_new_coordinate_on_axis.STL scale=0.001000 0.001000 0.001000
- link l_hip_roll: geometry collision box size=0.028500 0.046500 0.034000; visual mesh filename=meshes/XL-430_new_coordinate_on_axis.STL scale=0.001000 0.001000 0.001000
- link r_hip_pitch: geometry collision box size=0.028500 0.046500 0.034000; visual mesh filename=meshes/XL-430_new_coordinate_on_axis.STL scale=0.001000 0.001000 0.001000
- link r_hip_roll: geometry collision box size=0.028500 0.046500 0.034000; visual mesh filename=meshes/XL-430_new_coordinate_on_axis.STL scale=0.001000 0.001000 0.001000

File: model_generator_hrc/phonebot_general.urdf (robot description, URDF)
Before this commit: robot phonebot_general_6motor, 28 links, 27 joints
Links:
- link base_motor_link: geometry collision box size=0.028500 0.046500 0.034000; visual mesh filename=meshes/XL-430_new_coordinate_on_axis.STL scale=0.001000 0.001000 0.001000
- link l_ankle_pitch: geometry collision box size=0.028500 0.046500 0.034000; visual mesh filename=meshes/XL-430_new_coordinate_on_axis.STL scale=0.001000 0.001000 0.001000
- link l_ankle_roll: geometry collision box size=0.028500 0.046500 0.034000; visual mesh filename=meshes/XL-430_new_coordinate_on_axis.STL scale=0.001000 0.001000 0.001000
- link l_hip_calf: geometry collision box size=0.028500 0.046500 0.034000; visual mesh filename=meshes/XL-430_new_coordinate_on_axis.STL scale=0.001000 0.001000 0.001000
- link l_hip_pitch: geometry collision box size=0.028500 0.046500 0.034000; visual mesh filename=meshes/XL-430_new_coordinate_on_axis.STL scale=0.001000 0.001000 0.001000
- link l_hip_roll: geometry collision box size=0.028500 0.046500 0.034000; visual mesh filename=meshes/XL-430_new_coordinate_on_axis.STL scale=0.001000 0.001000 0.001000
- link l_hip_thigh: geometry collision box size=0.028500 0.046500 0.034000; visual mesh filename=meshes/XL-430_new_coordinate_on_axis.STL scale=0.001000 0.001000 0.001000
- link r_ankle_pitch: geometry collision box size=0.028500 0.046500 0.034000; visual mesh filename=meshes/XL-430_new_coordinate_on_axis.STL scale=0.001000 0.001000 0.001000
- link r_ankle_roll: geometry collision box size=0.028500 0.046500 0.034000; visual mesh filename=meshes/XL-430_new_coordinate_on_axis.STL scale=0.001000 0.001000 0.001000
- link r_hip_calf: geometry collision box size=0.028500 0.046500 0.034000; visual mesh filename=meshes/XL-430_new_coordinate_on_axis.STL scale=0.001000 0.001000 0.001000
- link r_hip_pitch: geometry collision box size=0.028500 0.046500 0.034000; visual mesh filename=meshes/XL-430_new_coordinate_on_axis.STL scale=0.001000 0.001000 0.001000
- link r_hip_roll: geometry collision box size=0.028500 0.046500 0.034000; visual mesh filename=meshes/XL-430_new_coordinate_on_axis.STL scale=0.001000 0.001000 0.001000
- link r_hip_thigh: geometry collision box size=0.028500 0.046500 0.034000; visual mesh filename=meshes/XL-430_new_coordinate_on_axis.STL scale=0.001000 0.001000 0.001000

Commit message: add damping to stabilize the motors

File: model_generator_hrc/chopstick_bot_general.urdf (robot description, URDF)
Before this commit: robot chopstick_bot, 12 links, 11 joints
Links:
- added link world
Joints:
- added joint world_to_base: type fixed, parent world, child base_motor_link, origin xyz=0.000000 0.000000 0.330000 rpy=0.000000 0.000000 0.000000

File: model_generator_hrc/phonebot_general.urdf (robot description, URDF)
Before this commit: robot phonebot_general_6motor, 28 links, 27 joints
Links:
- added link world
Joints:
- added joint world_to_base: type fixed, parent world, child base_motor_link, origin xyz=0.000000 0.000000 0.330000 rpy=0.000000 0.000000 0.000000

Commit message: add auto generate option cylinder_tip_box

File: model_generator_hrc/chopstick_bot_general.urdf (robot description, URDF)
Before this commit: robot chopstick_bot, 13 links, 12 joints
Links:
- link l_end_effector: geometry collision box size=0.020000 0.020000 0.020000; visual cylinder length=0.200000 radius=0.005000
- link r_end_effector: geometry collision box size=0.020000 0.020000 0.020000; visual cylinder length=0.200000 radius=0.005000
